File: _autosave-Peapod PCB.kicad_pcb (KiCad board)
At the start: 2 copper layers, 16 parts, among them J1 CONN_01X01, J2 CONN_01X02, J3 CONN_01X06, J5 CONN_01X01, J6 CONN_01X01, J7 CONN_01X02, U1 ESP8266

Commit message: stuff
Parts:
- added G***: LOGO, mod:LOGO, F.Cu at (215.9, 46.7)
- moved BTN2 12.5 mm to (160.3, 47.0)
- moved J1 1.52 mm to (165.6, 30.0)
Routing:
- net +3V3: track 108.4 -> 72.9 mm
- net Net-(BTN2-Pad2): track 19.1 -> 0.36 mm
- net Net-(J1-Pad1): track 14.1 -> 17.3 mm
- net GND: track 0.00 -> 0.21 mm, vias 0 -> 1
Other:
- board text added: "FSOSS 2017"
