File: Peapod PCB.kicad_pcb (KiCad board)
At the start: 2 copper layers, 70.9 x 26.9 mm, 20 parts, among them U1 ESP8266

Commit message: looks nice
Routing:
- net +3V3: track 118.9 -> 118.3 mm
Changed lines of the file:
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@@
     (thickness 1.6002)
     (drawings 7)
-    (tracks 122)
+    (tracks 125)
     (zones 0)
     (modules 20)
@@
     (effects (font (size 6 7) (thickness 0.3)) (justify mirror))
   )
+  (segment (start 187.706 33.21) (end 187.706 29.21) (width 0.635) (layer F.Cu) (net 1))
+  (segment (start 212.09 28.702) (end 212.09 33.02) (width 0.635) (layer F.Cu) (net 1) (status 800000))
+  (segment (start 211.328 27.94) (end 212.09 28.702) (width 0.635) (layer F.Cu) (net 1))
+  (segment (start 188.976 27.94) (end 211.328 27.94) (width 0.635) (layer F.Cu) (net 1))
+  (segment (start 187.706 29.21) (end 188.976 27.94) (width 0.635) (layer F.Cu) (net 1))
+  (segment (start 186.436 33.21) (end 187.706 33.21) (width 0.635) (layer F.Cu) (net 1))
+  (segment (start 187.706 33.21) (end 187.896 33.21) (width 0.635) (layer F.Cu) (net 1))
+  (segment (start 187.93 43.21) (end 185.42 43.21) (width 0.635) (layer F.Cu) (net 1) (status 800000))
+  (segment (start 188.722 42.418) (end 187.93 43.21) (width 0.635) (layer F.Cu) (net 1))
+  (segment (start 188.722 34.036) (end 188.722 42.418) (width 0.635) (layer F.Cu) (net 1))
+  (segment (start 187.896 33.21) (end 188.722 34.036) (width 0.635) (layer F.Cu) (net 1))
   (segment (start 156.34 39.37) (end 156.34 50.168) (width 0.635) (layer F.Cu) (net 1))
+  (segment (start 156.34 50.168) (end 157.226 51.054) (width 0.635) (layer F.Cu) (net 1))
+  (segment (start 157.226 51.054) (end 181.864 51.054) (width 0.635) (layer F.Cu) (net 1))
+  (segment (start 181.864 51.054) (end 183.388 49.53) (width 0.635) (layer F.Cu) (net 1))
+  (segment (start 183.388 49.53) (end 183.388 45.242) (width 0.635) (layer F.Cu) (net 1))
   (segment (start 183.388 45.242) (end 185.42 43.21) (width 0.635) (layer F.Cu) (net 1))
-  (segment (start 183.388 49.53) (end 183.388 45.242) (width 0.635) (layer F.Cu) (net 1))
-  (segment (start 181.864 51.054) (end 183.388 49.53) (width 0.635) (layer F.Cu) (net 1))
-  (segment (start 157.226 51.054) (end 181.864 51.054) (width 0.635) (layer F.Cu) (net 1))
-  (segment (start 156.34 50.168) (end 157.226 51.054) (width 0.635) (layer F.Cu) (net 1))
   (segment (start 185.39 43.21) (end 185.42 43.21) (width 0.635) (layer F.Cu) (net 1))
-  (segment (start 185.42 43.21) (end 187.93 43.21) (width 0.635) (layer F.Cu) (net 1))
-  (segment (start 187.96 35.75) (end 185.42 33.21) (width 0.635) (layer F.Cu) (net 1))
-  (segment (start 187.96 43.18) (end 187.96 35.75) (width 0.635) (layer F.Cu) (net 1))
-  (segment (start 187.93 43.21) (end 187.96 43.18) (width 0.635) (layer F.Cu) (net 1))
-  (segment (start 185.42 33.21) (end 186.5 33.21) (width 0.635) (layer F.Cu) (net 1))
-  (segment (start 212.09 27.94) (end 212.09 33.02) (width 0.635) (layer F.Cu) (net 1))
-  (segment (start 187.96 27.94) (end 212.09 27.94) (width 0.635) (layer F.Cu) (net 1))
-  (segment (start 187.96 31.75) (end 187.96 27.94) (width 0.635) (layer F.Cu) (net 1))
-  (segment (start 186.5 33.21) (end 187.96 31.75) (width 0.635) (layer F.Cu) (net 1))
+  (segment (start 185.42 33.21) (end 186.436 33.21) (width 0.635) (layer F.Cu) (net 1))
   (segment (start 207.09 40.64) (end 207.09 38.1) (width 0.635) (layer F.Cu) (net 1))
   (segment (start 207.09 38.1) (end 212.09 33.1) (width 0.635) (layer F.Cu) (net 1))
@@
   (segment (start 172.72 36.195) (end 176.45 36.195) (width 0.635) (layer F.Cu) (net 6))
   (segment (start 176.45 36.195) (end 177.72 37.465) (width 0.635) (layer F.Cu) (net 6))
-  (segment (start 182.372 30.988) (end 180.292 30.988) (width 0.635) (layer F.Cu) (net 7) (status 800000))
-  (segment (start 180.292 30.988) (end 178.768 29.464) (width 0.635) (layer F.Cu) (net 7) (status C00000))
-  (segment (start 185.42 35.21) (end 183.546 35.21) (width 0.635) (layer F.Cu) (net 7) (status C00000))
-  (segment (start 183.546 35.21) (end 182.372 34.036) (width 0.635) (layer F.Cu) (net 7) (status 400000))
+  (segment (start 182.372 30.988) (end 180.292 30.988) (width 0.635) (layer F.Cu) (net 7))
+  (segment (start 180.292 30.988) (end 178.768 29.464) (width 0.635) (layer F.Cu) (net 7))
+  (segment (start 185.42 35.21) (end 183.546 35.21) (width 0.635) (layer F.Cu) (net 7))
+  (segment (start 183.546 35.21) (end 182.372 34.036) (width 0.635) (layer F.Cu) (net 7))
   (via (at 182.372 34.036) (size 0.6858) (drill 0.3302) (layers F.Cu B.Cu) (net 7))
   (segment (start 182.372 34.036) (end 182.372 30.988) (width 0.635) (layer B.Cu) (net 7))
   (via (at 182.372 30.988) (size 0.6858) (drill 0.3302) (layers F.Cu B.Cu) (net 7))
-  (segment (start 182.372 30.988) (end 184.15 29.21) (width 0.635) (layer F.Cu) (net 7) (status 800000))
-  (segment (start 184.15 29.21) (end 185.42 29.21) (width 0.635) (layer F.Cu) (net 7) (status C00000))
+  (segment (start 182.372 30.988) (end 184.15 29.21) (width 0.635) (layer F.Cu) (net 7))
+  (segment (start 184.15 29.21) (end 185.42 29.21) (width 0.635) (layer F.Cu) (net 7))
   (segment (start 213.36 50.292) (end 213.36 48.768) (width 0.635) (layer F.Cu) (net 9))
   (segment (start 213.36 48.768) (end 209.296 43.688) (width 0.635) (layer F.Cu) (net 9))
@@
   (segment (start 207.264 35.306) (end 203.2 35.306) (width 0.635) (layer F.Cu) (net 9))
   (segment (start 207.01 31.242) (end 211.074 31.242) (width 0.635) (layer F.Cu) (net 10))
-  (segment (start 219.71 42.672) (end 219.71 50.292) (width 0.635) (layer F.Cu) (net 10) (status 800000))
+  (segment (start 219.71 42.672) (end 219.71 50.292) (width 0.635) (layer F.Cu) (net 10))
   (segment (start 217.17 40.132) (end 219.71 42.672) (width 0.635) (layer F.Cu) (net 10))
   (segment (start 217.17 38.608) (end 217.17 40.132) (width 0.635) (layer F.Cu) (net 10))
@@
   (segment (start 211.074 31.242) (end 213.106 31.242) (width 0.635) (layer B.Cu) (net 10))
   (via (at 211.074 31.242) (size 0.6858) (drill 0.3302) (layers F.Cu B.Cu) (net 10))
-  (segment (start 207.01 33.02) (end 207.01 31.242) (width 0.635) (layer F.Cu) (net 10) (status 400000))
-  (segment (start 204.978 29.21) (end 199.42 29.21) (width 0.635) (layer F.Cu) (net 10) (status 800000))
+  (segment (start 207.01 33.02) (end 207.01 31.242) (width 0.635) (layer F.Cu) (net 10))
+  (segment (start 204.978 29.21) (end 199.42 29.21) (width 0.635) (layer F.Cu) (net 10))
   (segment (start 207.01 31.242) (end 204.978 29.21) (width 0.635) (layer F.Cu) (net 10))
   (segment (start 187.198 50.292) (end 187.198 47.498) (width 0.635) (layer F.Cu) (net 12))
@@
   (segment (start 196.438 35.21) (end 196.088 35.56) (width 0.635) (layer F.Cu) (net 13))
   (segment (start 196.088 48.768) (end 194.564 50.292) (width 0.635) (layer F.Cu) (net 13))
-  (segment (start 199.42 37.21) (end 203.5 37.21) (width 0.635) (layer F.Cu) (net 14) (status 400000))
-  (segment (start 203.5 37.21) (end 204.39 38.1) (width 0.635) (layer F.Cu) (net 14) (status 800000))
+  (segment (start 199.42 37.21) (end 203.5 37.21) (width 0.635) (layer F.Cu) (net 14))
+  (segment (start 203.5 37.21) (end 204.39 38.1) (width 0.635) (layer F.Cu) (net 14))
   (segment (start 207.216 50.546) (end 207.216 48.72) (width 0.635) (layer F.Cu) (net 14))
   (segment (start 207.216 48.72) (end 205.74 45.72) (width 0.635) (layer F.Cu) (net 14))
